File: hardware/LED_Stem.kicad_sch (KiCad schematic)
At the start: 4 parts

Commit message: first commit with github actions
Parts:
- D2, D3: Package 4014 -> 3014
Changed lines of the file:
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@@
       (effects (font (size 1.27 1.27)) hide)
     )
-    (property "Package" "4014" (id 5) (at 50.8 66.04 0)
+    (property "Package" "3014" (id 5) (at 50.8 66.04 0)
       (effects (font (size 1.27 1.27)) hide)
     )
@@
       (effects (font (size 1.27 1.27)) hide)
     )
-    (property "Package" "4014" (id 5) (at 63.5 66.04 0)
+    (property "Package" "3014" (id 5) (at 63.5 66.04 0)
       (effects (font (size 1.27 1.27)) hide)
     )
